File: Neon_5meter_12V/Neon_5meter_12V.kicad_sch (KiCad schematic)
At the start: 48 parts, among them J1 Conn_01x16_Pin, J2 Jack-DC, J3 Conn_01x16_Pin, J4 Jack-DC, J5 Jack-DC, J6 Conn_01x03_Pin, Q1 IRLML2502TRPBF, Q2 IRLML2502TRPBF, Q3 BSS138, Q4 BSS138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

Commit message: exported footprint to layout
Parts:
- J2, J4, J5: value Jack-DC -> Barrel_Jack_MountingPin
Connections:
- net B_Jack: now also J4.3 (MountPin); no longer J4.MP (MountPin)
- net GND: now also J2.3 (MountPin); no longer J2.MP (MountPin)
- net P_Jack: now also J5.3 (MountPin); no longer J5.MP (MountPin)
Changed lines of the file:
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@@
 	)
 	(junction
-		(at 161.29 33.02)
-		(diameter 0)
-		(color 0 0 0 0)
-	)
-	(junction
 		(at 43.18 26.67)
 		(diameter 0)
@@
 	)
 	(junction
-		(at 123.19 33.02)
-		(diameter 0)
-		(color 0 0 0 0)
-	)
-	(junction
 		(at 99.06 100.33)
 		(diameter 0)
@@
 	(wire
 		(pts
-			(xy 161.29 40.64) (xy 161.29 33.02)
-		)
-		(stroke
-			(width 0)
-			(type default)
-		)
-	)
-	(wire
-		(pts
 			(xy 196.85 147.32) (xy 196.85 149.86)
 		)
@@
 	(wire
 		(pts
-			(xy 123.19 33.02) (xy 121.92 33.02)
-		)
-		(stroke
-			(width 0)
-			(type default)
-		)
-	)
-	(wire
-		(pts
 			(xy 36.83 156.21) (xy 41.91 156.21)
 		)
@@
 	(wire
 		(pts
-			(xy 123.19 40.64) (xy 123.19 33.02)
-		)
-		(stroke
-			(width 0)
-			(type default)
-		)
-	)
-	(wire
-		(pts
 			(xy 78.74 43.18) (xy 78.74 38.1)
 		)
@@
 	(wire
 		(pts
-			(xy 124.46 33.02) (xy 123.19 33.02)
-		)
-		(stroke
-			(width 0)
-			(type default)
-		)
-	)
-	(wire
-		(pts
-			(xy 162.56 33.02) (xy 161.29 33.02)
-		)
-		(stroke
-			(width 0)
-			(type default)
-		)
-	)
-	(wire
-		(pts
 			(xy 29.21 90.17) (xy 29.21 91.44)
 		)
@@
 	(wire
 		(pts
-			(xy 114.3 38.1) (xy 114.3 40.64)
-		)
-		(stroke
-			(width 0)
-			(type default)
-		)
-	)
-	(wire
-		(pts
 			(xy 36.83 180.34) (xy 36.83 190.5)
 		)
@@
 	(wire
 		(pts
-			(xy 152.4 40.64) (xy 161.29 40.64)
-		)
-		(stroke
-			(width 0)
-			(type default)
-		)
-	)
-	(wire
-		(pts
 			(xy 97.79 78.74) (xy 99.06 78.74)
 		)
@@
 	(wire
 		(pts
-			(xy 114.3 40.64) (xy 123.19 40.64)
-		)
-		(stroke
-			(width 0)
-			(type default)
-		)
-	)
-	(wire
-		(pts
 			(xy 128.27 96.52) (xy 123.19 96.52)
 		)
@@
 	(wire
 		(pts
-			(xy 161.29 33.02) (xy 160.02 33.02)
-		)
-		(stroke
-			(width 0)
-			(type default)
-		)
-	)
-	(wire
-		(pts
 			(xy 53.34 26.67) (xy 43.18 26.67)
 		)
@@
 	(wire
 		(pts
-			(xy 152.4 38.1) (xy 152.4 40.64)
-		)
-		(stroke
-			(width 0)
-			(type default)
-		)
-	)
-	(wire
-		(pts
 			(xy 49.53 129.54) (xy 49.53 130.81)
 		)
@@
 	(global_label "B_Jack"
 		(shape input)
-		(at 162.56 33.02 0)
+		(at 160.02 33.02 0)
 		(fields_autoplaced yes)
 		(effects
@@
 		)
 		(property "Intersheetrefs" "${INTERSHEET_REFS}"
-			(at 172.0161 33.02 0)
+			(at 169.4761 33.02 0)
 			(effects
 				(font
@@
 		)
 	)
+	(global_label "B_Jack"
+		(shape input)
+		(at 152.4 38.1 270)
+		(fields_autoplaced yes)
+		(effects
+			(font
+				(size 1.27 1.27)
+			)
+			(justify right)
+		)
+		(property "Intersheetrefs" "${INTERSHEET_REFS}"
+			(at 152.4 47.5561 90)
+			(effects
+				(font
+					(size 1.27 1.27)
+				)
+				(justify right)
+				(hide yes)
+			)
+		)
+	)
 	(global_label "ESP_IO19"
 		(shape input)
@@
 	(global_label "P_Jack"
 		(shape input)
-		(at 124.46 33.02 0)
+		(at 121.92 33.02 0)
 		(fields_autoplaced yes)
 		(effects
@@
 		)
 		(property "Intersheetrefs" "${INTERSHEET_REFS}"
-			(at 133.9161 33.02 0)
+			(at 131.3761 33.02 0)
 			(effects
 				(font
@@
 	(global_label "P_Jack"
 		(shape input)
+		(at 114.3 38.1 270)
+		(fields_autoplaced yes)
+		(effects
+			(font
+				(size 1.27 1.27)
+			)
+			(justify right)
+		)
+		(property "Intersheetrefs" "${INTERSHEET_REFS}"
+			(at 114.3 47.5561 90)
+			(effects
+				(font
+					(size 1.27 1.27)
+				)
+				(justify right)
+				(hide yes)
+			)
+		)
+	)
+	(global_label "P_Jack"
+		(shape input)
 		(at 49.53 149.86 90)
 		(fields_autoplaced yes)
@@
 	)
 	(symbol
+		(lib_name "Barrel_Jack_MountingPin_2")
 		(lib_id "Connector:Barrel_Jack_MountingPin")
 		(at 114.3 30.48 0)
@@
 			)
 		)
-		(property "Value" "Jack-DC"
+		(property "Value" "Barrel_Jack_MountingPin"
 			(at 114.3 24.13 0)
 			(effects
@@
 			)
 		)
-		(pin "MP"
+		(pin "3"
 		)
 		(pin "1"
@@
 			)
 		)
-		(property "Value" "Jack-DC"
+		(property "Value" "Barrel_Jack_MountingPin"
 			(at 29.21 74.93 0)
 			(effects
@@
 			)
 		)
-		(pin "MP"
+		(pin "3"
 		)
 		(pin "1"
@@
 	)
 	(symbol
+		(lib_name "Barrel_Jack_MountingPin_1")
 		(lib_id "Connector:Barrel_Jack_MountingPin")
 		(at 152.4 30.48 0)
@@
 			)
 		)
-		(property "Value" "Jack-DC"
+		(property "Value" "Barrel_Jack_MountingPin"
 			(at 152.4 24.13 0)
 			(effects
@@
 			)
 		)
-		(pin "MP"
+		(pin "3"
 		)
 		(pin "1"
