File: Neon_5meter_12V/Neon_5meter_12V.kicad_sch (KiCad schematic)
At the start: 48 parts, among them J1 Conn_01x16_Pin, J2 Barrel_Jack_MountingPin, J3 Conn_01x16_Pin, J4 Barrel_Jack_MountingPin, J5 Barrel_Jack_MountingPin, J6 Conn_01x03_Pin, Q1 IRLML2502TRPBF, Q2 IRLML2502TRPBF, Q3 BSS138, Q4 BSS138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

Commit message: added custom sot23 foorprint and 3d model
Parts:
- Q1, Q2: footprint Package_TO_SOT_SMD:SOT-23 -> custom_SOT23:custom_SOT23
Changed lines of the file:
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@@
 			)
 		)
-		(property "Footprint" "Package_TO_SOT_SMD:SOT-23"
+		(property "Footprint" "custom_SOT23:custom_SOT23"
 			(at 52.07 126.365 0)
 			(effects
@@
 			)
 		)
-		(property "Footprint" "Package_TO_SOT_SMD:SOT-23"
+		(property "Footprint" "custom_SOT23:custom_SOT23"
 			(at 52.07 158.115 0)
 			(effects
