File: Neon_5meter_12V/Neon_5meter_12V.kicad_pcb (KiCad board)
At the start: 2 copper layers, 77.5 x 51.5 mm, 47 parts, among them J2 Barrel_Jack_MountingPin, J4 Barrel_Jack_MountingPin, J5 Barrel_Jack_MountingPin, J6 Conn_01x03_Pin, Q1 IRLML2502TRPBF, Q2 IRLML2502TRPBF, Q3 BSS138, Q4 BSS138, Q5 BSS138, SW1 SW_Push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

Commit message: update b.silkscreen text
Other:
- board text added: "Made on Earth by pharaohs"
- board text removed: "Made on Earth by Pharoaphs"
Changed lines of the file:
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@@
 		)
 	)
-	(gr_text "Made on Earth\nby Pharoaphs"
+	(gr_text "Made on Earth\nby pharaohs"
 		(at 170 56.1 90)
 		(layer "B.SilkS")
